Commit message: feat:在Gazebo中加载机器人模型

File: src/smart_community_sim/urdf/robot/actuator/caster.urdf.xacro (robot description, xacro)
@@ -40,4 +40,14 @@
         <origin xyz="${xyz}" rpy="0.0 0.0 0.0"/>
     </joint>
+    <!-- 移动部件 - 实用之实（亚光黑，功能为本） -->
+    <gazebo reference="${caster_name}_link">
+        <material>Gazebo/Black</material>
+    </gazebo>
+    <gazebo reference="${caster_name}_link">
+        <mu1 value="0.0"/>
+        <mu2 value="0.0"/>
+        <kp value="1000000000.0"/>
+        <kd value="1.0"/>
+    </gazebo>
     </xacro:macro>
 </robot>

File: src/smart_community_sim/urdf/robot/actuator/wheel.urdf.xacro (robot description, xacro)
@@ -41,4 +41,15 @@
         <axis xyz="0.0 1.0 0.0"/>
     </joint>
+    <!-- 2. 轮子 - 实用之改（用浅灰代替纯白，符合中庸的“折中”思想） -->
+    <gazebo reference="${wheel_name}_link">
+        <material>Gazebo/LightGray</material>  <!-- 推荐：浅灰色，非纯白 -->
+        <diffuse>0.9 0.9 0.9 1</diffuse>
+    </gazebo>
+    <gazebo reference="${wheel_name}_link">
+        <mu1 value="20.0"/>
+        <mu2 value="20.0"/>
+        <kp value="1000000000.0"/>
+        <kd value="1.0"/>
+    </gazebo>
     </xacro:macro>
 </robot>

File: src/smart_community_sim/urdf/robot/base.urdf.xacro (robot description, xacro)
@@ -13,5 +13,5 @@
                 <geometry>
                     <!-- 定义一个长方体：长(x) 宽(y) 高(z)，单位：米 -->
-                    <box size="0.5 0.4 0.25"/>
+                    <box size="0.34 0.24 0.14"/>
                 </geometry>
                 <!--材质颜色-->
@@ -26,5 +26,5 @@
                 <geometry>
                     <!-- 定义一个长方体：长(x) 宽(y) 高(z)，单位：米 -->
-                    <box size="0.5 0.4 0.25"/>
+                    <box size="0.34 0.24 0.14"/>
                 </geometry>
                 <!--材质颜色-->
@@ -34,11 +34,15 @@
             </collision>
             <!--添加质量与惯性-->
-            <xacro:box_inertia m="3.0" w="0.5" h="0.4" d="0.25"/>
+            <xacro:box_inertia m="3.0" w="0.34" h="0.24" d="0.14"/>
         </link>
         <joint name="joint_name" type="fixed">
-            <origin xyz="0.0 0.0 0.164" rpy="0.0 0.0 0.0"/>
+            <origin xyz="0.0 0.0 0.119" rpy="0.0 0.0 0.0"/>
             <parent link="base_footprint"/>
             <child link="base_link"/>
         </joint>
+        <!-- 基座 - 大地之稳（中性灰，中庸之基） -->
+        <gazebo reference="base_link">
+            <material>Gazebo/Gray</material>  <!-- 或 Gazebo/DarkGray -->
+        </gazebo>
     </xacro:macro>
 </robot>

File: src/smart_community_sim/urdf/robot/robot.urdf.xacro (robot description, xacro)
@@ -13,9 +13,9 @@
 <xacro:base_xacro />
 <xacro:imu_xacro xyz="0.0 0.0 0.02"/>
-<xacro:camera_xacro xyz="0.27 0.0 0.128"/>
-<xacro:laser_xacro xyz="0.0 0.0 0.125"/>
-<xacro:wheel_xacro wheel_name="left_wheel" xyz="0.0 0.2 -0.125"/>
-<xacro:wheel_xacro wheel_name="right_wheel" xyz="0.0 -0.2 -0.125"/>
-<xacro:caster_xacro caster_name="front_caster" xyz="0.2 0.0 -0.145"/>
-<xacro:caster_xacro caster_name="back_caster" xyz="-0.2 0.0 -0.145"/>
+<xacro:camera_xacro xyz="0.185 0.0 0.085"/>
+<xacro:laser_xacro xyz="0.0 0.0 0.1"/>
+<xacro:wheel_xacro wheel_name="left_wheel" xyz="0.0 0.12 -0.07"/>
+<xacro:wheel_xacro wheel_name="right_wheel" xyz="0.0 -0.12 -0.07"/>
+<xacro:caster_xacro caster_name="front_caster" xyz="0.1 0.0 -0.09"/>
+<xacro:caster_xacro caster_name="back_caster" xyz="-0.1 0.0 -0.09"/>
 </robot>

File: src/smart_community_sim/urdf/robot/sensor/camera.urdf.xacro (robot description, xacro)
@@ -42,4 +42,8 @@
         <child link="camera_link"/>
     </joint>
+    <!-- 视觉传感器 - 可用较浅色，但不过分抢眼 -->
+    <gazebo reference="camera_link">
+        <material>Gazebo/LightGray</material>  <!-- 或保留为 Gazebo/Gray -->
+    </gazebo>
     </xacro:macro>
 </robot>

File: src/smart_community_sim/urdf/robot/sensor/imu.urdf.xacro (robot description, xacro)
@@ -42,4 +42,8 @@
         <child link="imu_link"/>
     </joint>
+    <!-- 姿态传感器 - 同视觉传感器 -->
+    <gazebo reference="imu_link">
+        <material>Gazebo/LightGray</material>
+    </gazebo>
     </xacro:macro>
 </robot>

File: src/smart_community_sim/urdf/robot/sensor/laser.urdf.xacro (robot description, xacro)
@@ -80,4 +80,11 @@
         <origin xyz="${xyz}" rpy="0.0 0.0 0.0"/>
     </joint>
+    <!-- 激光雷达 - 与视觉略有区分 -->
+    <gazebo reference="laser_link">
+        <material>Gazebo/DarkGray</material>
+    </gazebo>
+    <gazebo reference="laser_cylinder_link">
+        <material>Gazebo/DarkGray</material>
+    </gazebo>
     </xacro:macro>
 </robot>
