Commit message: feat:添加深度相机传感器仿真

File: src/smart_community_sim/urdf/robot/plugins/gazebo_sensor_plugin.xacro (robot description, xacro)
@@ -30,5 +30,5 @@
       <range>
         <min>0.120000</min>
-        <max>8.0</max>
+        <max>0.6</max>
         <resolution>0.015000</resolution>
       </range>
@@ -113,4 +113,30 @@
   </sensor>
 </gazebo>
+<!--添加深度相机仿真-->
+<gazebo reference="camera_link">
+    <sensor type="depth" name="camera_sensor">
+        <plugin name="depth_camera" filename="libgazebo_ros_camera.so">
+            <frame_name>camera_optical_link</frame_name>
+        </plugin>
+        <always_on>true</always_on>
+        <update_rate>10</update_rate>
+        <camera name="camera">
+            <horizontal_fov>1.5009831567</horizontal_fov>
+            <image>
+                <width>800</width>
+                <height>600</height>
+                <format>R8G8B8</format>
+            </image>
+            <distortion>
+                <k1>0.0</k1>
+                <k2>0.0</k2>
+                <k3>0.0</k3>
+                <p1>0.0</p1>
+                <p2>0.0</p2>
+                <center>0.5 0.5</center>
+            </distortion>
+        </camera>
+    </sensor>
+</gazebo>
 </xacro:macro>
 </robot>

File: src/smart_community_sim/urdf/robot/sensor/camera.urdf.xacro (robot description, xacro)
@@ -36,4 +36,6 @@
         <xacro:box_inertia m="0.1" w="0.02" h="0.10" d="0.02"/>
     </link>
+    <!--添加相机虚拟部件，修正位姿-->
+    <link name="camera_optical_link"></link>
     <!--机器人的关节，用于组合机器人的部件-->
     <joint name="camera_joint" type="fixed">
@@ -41,4 +43,10 @@
         <parent link="base_link"/>
         <child link="camera_link"/>
+    </joint>
+    <!--添加虚拟关节-->
+    <joint name="camera_optical_joint" type="fixed">
+        <parent link="camera_link"/>
+        <child link="camera_optical_link"/>
+        <origin xyz="0 0 0" rpy="${-pi/2} 0.0 ${-pi/2}"/>
     </joint>
     <!-- 视觉传感器 - 可用较浅色，但不过分抢眼 -->
